Commit message: change forward to back climb

File: dancer_urdf_model/robots/dancer_urdf_model.xacro (robot description, xacro)
@@ -4,4 +4,5 @@
   <xacro:property name="dam" value="0.0"/>
   <xacro:property name="fri" value="10.0"/>
+  <xacro:property name="mass_multi" value="1.0"/>
 <!-- root link -->
   <link
@@ -21,5 +22,5 @@
         rpy="0 0 0" />
       <mass
-        value="0.66907" />
+        value="${0.66907 * mass_multi}" />
       <inertia
         ixx="0.004463976"
@@ -61,5 +62,5 @@
         rpy="0 0 0" />
       <mass
-        value="0.0560380421735799" />
+        value="${0.0560380421735799 * mass_multi}" />
       <inertia
         ixx="6.80542660516315E-06"
@@ -117,5 +118,5 @@
         rpy="0 0 0" />
       <mass
-        value="0.067365" />
+        value="${0.067365 * mass_multi}" />
       <inertia
         ixx="2.0873E-05"
@@ -173,5 +174,5 @@
         rpy="0 0 0" />
       <mass
-        value="0.142976459032186" />
+        value="${0.142976459032186 * mass_multi}" />
       <inertia
         ixx="2.49420588469075E-04"
@@ -229,5 +230,5 @@
         rpy="0 0 0" />
       <mass
-        value="0.021948273112724" />
+        value="${0.021948273112724 * mass_multi}" />
       <inertia
         ixx="1.788488E-04"
@@ -285,5 +286,5 @@
         rpy="0 0 0" />
       <mass
-        value="0.141656759847187" />
+        value="${0.141656759847187 * mass_multi}" />
       <inertia
         ixx="2.44964545549609E-04"
@@ -341,5 +342,5 @@
         rpy="0 0 0" />
       <mass
-        value="0.021948273112724" />
+        value="${0.021948273112724 * mass_multi}" />
       <inertia
         ixx="1.442092E-04"
@@ -397,5 +398,5 @@
         rpy="0 0 0" />
       <mass
-        value="0.220741166410594" />
+        value="${0.220741166410594 * mass_multi}" />
       <inertia
         ixx="8.47561E-04"
@@ -453,5 +454,5 @@
         rpy="0 0 0" />
       <mass
-        value="0.0513468076618724" />
+        value="${0.0513468076618724 * mass_multi}" />
       <inertia
         ixx="3.0932E-05"
@@ -509,5 +510,5 @@
         rpy="0 0 0" />
       <mass
-        value="0.178226116015845" />
+        value="${0.178226116015845 * mass_multi}" />
       <inertia
         ixx="1.44373E-04"
@@ -565,5 +566,5 @@
         rpy="0 0 0" />
       <mass
-        value="0.117898503490257" />
+        value="${0.117898503490257 * mass_multi}" />
       <inertia
         ixx="1.493574E-03"
@@ -621,5 +622,5 @@
         rpy="0 0 0" />
       <mass
-        value="0.0278306854029525" />
+        value="${0.0278306854029525 * mass_multi}" />
       <inertia
         ixx="1.48269E-04"
@@ -677,5 +678,5 @@
         rpy="0 0 0" />
       <mass
-        value="0.177450614870689" />
+        value="${0.177450614870689 * mass_multi}" />
       <inertia
         ixx="3.75156E-04"
@@ -733,5 +734,5 @@
         rpy="0 0 0" />
       <mass
-        value="0.13465253780049" />
+        value="${0.13465253780049 * mass_multi}" />
       <inertia
         ixx="6.9952E-04"
@@ -789,5 +790,5 @@
         rpy="0 0 0" />
       <mass
-        value="0.0513468076618724" />
+        value="${0.0513468076618724 * mass_multi}" />
       <inertia
         ixx="3.6027E-05"
@@ -845,5 +846,5 @@
         rpy="0 0 0" />
       <mass
-        value="0.178226118022815" />
+        value="${0.178226118022815 * mass_multi}" />
       <inertia
         ixx="1.44373E-04"
@@ -901,5 +902,5 @@
         rpy="0 0 0" />
       <mass
-        value="0.117898502766572" />
+        value="${0.117898502766572 * mass_multi}" />
       <inertia
         ixx="1.493573E-03"
@@ -957,5 +958,5 @@
         rpy="0 0 0" />
       <mass
-        value="0.0278306854029525" />
+        value="${0.0278306854029525 * mass_multi}" />
       <inertia
         ixx="1.48269E-04"
@@ -1013,5 +1014,5 @@
         rpy="0 0 0" />
       <mass
-        value="0.177450615338578" />
+        value="${0.177450615338578 * mass_multi}" />
       <inertia
         ixx="3.75156E-04"
@@ -1069,5 +1070,5 @@
         rpy="0 0 0" />
       <mass
-        value="0.133904507779755" />
+        value="${0.133904507779755 * mass_multi}" />
       <inertia
         ixx="6.95451E-04"
@@ -1126,5 +1127,5 @@
         rpy="0 -1.5708 0" />
       <mass
-        value="0.00912844677087833" />
+        value="${0.00912844677087833 * mass_multi}" />
       <inertia
         ixx="0"
@@ -1177,4 +1178,5 @@
     <mu2>0.2</mu2>
     <material>Gazebo/Gray</material>
+    <gravity>true</gravity>
     <!--<turnGravityoff>false</turnGravityoff>-->
   </gazebo>
@@ -1183,4 +1185,5 @@
     <mu2>0.2</mu2>
     <material>Gazebo/Green</material>
+    <gravity>true</gravity>
     <!--<turnGravityoff>false</turnGravityoff>-->
   </gazebo>
@@ -1189,4 +1192,5 @@
     <mu2>0.2</mu2>
     <material>Gazebo/Green</material>
+    <gravity>true</gravity>
     <!--<turnGravityoff>false</turnGravityoff>-->
   </gazebo>
@@ -1195,4 +1199,5 @@
     <mu2>0.2</mu2>
     <material>Gazebo/Blue</material>
+    <gravity>true</gravity>
     <!--<turnGravityoff>false</turnGravityoff>-->
   </gazebo>
@@ -1201,4 +1206,5 @@
     <mu2>0.2</mu2>
     <material>Gazebo/Orange</material>
+    <gravity>true</gravity>
     <!--<turnGravityoff>false</turnGravityoff>-->
   </gazebo>
@@ -1207,4 +1213,5 @@
     <mu2>0.2</mu2>
     <material>Gazebo/Blue</material>
+    <gravity>true</gravity>
     <!--<turnGravityoff>false</turnGravityoff>-->
   </gazebo>
@@ -1213,4 +1220,5 @@
     <mu2>0.2</mu2>
     <material>Gazebo/Orange</material>
+    <gravity>true</gravity>
     <!--<turnGravityoff>false</turnGravityoff>-->
   </gazebo>
@@ -1219,4 +1227,5 @@
     <mu2>0.2</mu2>
     <material>Gazebo/Green</material>
+    <gravity>true</gravity>
     <!--<turnGravityoff>false</turnGravityoff>-->
   </gazebo>
@@ -1225,4 +1234,5 @@
     <mu2>0.2</mu2>
     <material>Gazebo/Black</material>
+    <gravity>true</gravity>
     <!--<turnGravityoff>false</turnGravityoff>-->
   </gazebo>
@@ -1231,4 +1241,5 @@
     <mu2>0.2</mu2>
     <material>Gazebo/Black</material>
+    <gravity>true</gravity>
     <!--<turnGravityoff>false</turnGravityoff>-->
   </gazebo>
@@ -1237,4 +1248,5 @@
     <mu2>0.2</mu2>
     <material>Gazebo/Blue</material>
+    <gravity>true</gravity>
     <!--<turnGravityoff>false</turnGravityoff>-->
   </gazebo>
@@ -1243,4 +1255,5 @@
     <mu2>0.2</mu2>
     <material>Gazebo/Orange</material>
+    <gravity>true</gravity>
     <!--<turnGravityoff>false</turnGravityoff>-->
   </gazebo>
@@ -1249,4 +1262,5 @@
     <mu2>0.2</mu2>
     <material>Gazebo/Blue</material>
+    <gravity>true</gravity>
     <!--<turnGravityoff>false</turnGravityoff>-->
   </gazebo>
@@ -1255,4 +1269,5 @@
     <mu2>0.2</mu2>
     <material>Gazebo/Orange</material>
+    <gravity>true</gravity>
     <!--<turnGravityoff>false</turnGravityoff>-->
   </gazebo>
@@ -1261,4 +1276,5 @@
     <mu2>0.2</mu2>
     <material>Gazebo/Black</material>
+    <gravity>true</gravity>
     <!--<turnGravityoff>false</turnGravityoff>-->
   </gazebo>
@@ -1267,4 +1283,5 @@
     <mu2>0.2</mu2>
     <material>Gazebo/Black</material>
+    <gravity>true</gravity>
     <!--<turnGravityoff>false</turnGravityoff>-->
   </gazebo>
@@ -1273,4 +1290,5 @@
     <mu2>0.2</mu2>
     <material>Gazebo/Black</material>
+    <gravity>true</gravity>
     <!--<turnGravityoff>false</turnGravityoff>-->
   </gazebo>
@@ -1279,4 +1297,5 @@
     <mu2>0.2</mu2>
     <material>Gazebo/Black</material>
+    <gravity>true</gravity>
     <!--<turnGravityoff>false</turnGravityoff>-->
   </gazebo>
@@ -1285,4 +1304,5 @@
     <mu2>0.2</mu2>
      <material>Gazebo/Black</material>
+    <gravity>true</gravity>
     <!--<turnGravityoff>false</turnGravityoff>-->
   </gazebo>
@@ -1291,4 +1311,5 @@
     <mu2>0.2</mu2>
     <material>Gazebo/Black</material>
+    <gravity>true</gravity>
     <!--<turnGravityoff>false</turnGravityoff>-->
   </gazebo>
@@ -1297,5 +1318,4 @@
     <mu2>0.2</mu2>
     <material>Gazebo/Red</material>
-    <!--<turnGravityoff>false</turnGravityoff>-->
     <sensor type="camera" name="camera1">
       <always_on>true</always_on>

Commit message: change frition and mass of body and PID

File: dancer_urdf_model/robots/dancer_urdf_model.xacro (robot description, xacro)
@@ -4,5 +4,6 @@
   <xacro:property name="dam" value="0.0"/>
   <xacro:property name="fri" value="10.0"/>
-  <xacro:property name="mass_multi" value="1.0"/>
+  <xacro:property name="mass_upper" value="0.4"/>
+  <xacro:property name="mass_lower" value="2.0"/>
 <!-- root link -->
   <link
@@ -22,5 +23,5 @@
         rpy="0 0 0" />
       <mass
-        value="${0.66907 * mass_multi}" />
+        value="${0.66907 * mass_upper}" />
       <inertia
         ixx="0.004463976"
@@ -62,5 +63,5 @@
         rpy="0 0 0" />
       <mass
-        value="${0.0560380421735799 * mass_multi}" />
+        value="${0.0560380421735799 * mass_upper}" />
       <inertia
         ixx="6.80542660516315E-06"
@@ -118,5 +119,5 @@
         rpy="0 0 0" />
       <mass
-        value="${0.067365 * mass_multi}" />
+        value="${0.067365 * mass_upper}" />
       <inertia
         ixx="2.0873E-05"
@@ -174,5 +175,5 @@
         rpy="0 0 0" />
       <mass
-        value="${0.142976459032186 * mass_multi}" />
+        value="${0.142976459032186 * mass_upper}" />
       <inertia
         ixx="2.49420588469075E-04"
@@ -230,5 +231,5 @@
         rpy="0 0 0" />
       <mass
-        value="${0.021948273112724 * mass_multi}" />
+        value="${0.021948273112724 * mass_upper}" />
       <inertia
         ixx="1.788488E-04"
@@ -286,5 +287,5 @@
         rpy="0 0 0" />
       <mass
-        value="${0.141656759847187 * mass_multi}" />
+        value="${0.141656759847187 * mass_upper}" />
       <inertia
         ixx="2.44964545549609E-04"
@@ -342,5 +343,5 @@
         rpy="0 0 0" />
       <mass
-        value="${0.021948273112724 * mass_multi}" />
+        value="${0.021948273112724 * mass_upper}" />
       <inertia
         ixx="1.442092E-04"
@@ -398,5 +399,5 @@
         rpy="0 0 0" />
       <mass
-        value="${0.220741166410594 * mass_multi}" />
+        value="${0.220741166410594 * mass_upper}" />
       <inertia
         ixx="8.47561E-04"
@@ -454,5 +455,5 @@
         rpy="0 0 0" />
       <mass
-        value="${0.0513468076618724 * mass_multi}" />
+        value="${0.0513468076618724 * mass_lower}" />
       <inertia
         ixx="3.0932E-05"
@@ -510,5 +511,5 @@
         rpy="0 0 0" />
       <mass
-        value="${0.178226116015845 * mass_multi}" />
+        value="${0.178226116015845 * mass_lower}" />
       <inertia
         ixx="1.44373E-04"
@@ -566,5 +567,5 @@
         rpy="0 0 0" />
       <mass
-        value="${0.117898503490257 * mass_multi}" />
+        value="${0.117898503490257 * mass_lower}" />
       <inertia
         ixx="1.493574E-03"
@@ -622,5 +623,5 @@
         rpy="0 0 0" />
       <mass
-        value="${0.0278306854029525 * mass_multi}" />
+        value="${0.0278306854029525 * mass_lower}" />
       <inertia
         ixx="1.48269E-04"
@@ -678,5 +679,5 @@
         rpy="0 0 0" />
       <mass
-        value="${0.177450614870689 * mass_multi}" />
+        value="${0.177450614870689 * mass_lower}" />
       <inertia
         ixx="3.75156E-04"
@@ -734,5 +735,5 @@
         rpy="0 0 0" />
       <mass
-        value="${0.13465253780049 * mass_multi}" />
+        value="${0.13465253780049 * mass_lower}" />
       <inertia
         ixx="6.9952E-04"
@@ -790,5 +791,5 @@
         rpy="0 0 0" />
       <mass
-        value="${0.0513468076618724 * mass_multi}" />
+        value="${0.0513468076618724 * mass_lower}" />
       <inertia
         ixx="3.6027E-05"
@@ -846,5 +847,5 @@
         rpy="0 0 0" />
       <mass
-        value="${0.178226118022815 * mass_multi}" />
+        value="${0.178226118022815 * mass_lower}" />
       <inertia
         ixx="1.44373E-04"
@@ -902,5 +903,5 @@
         rpy="0 0 0" />
       <mass
-        value="${0.117898502766572 * mass_multi}" />
+        value="${0.117898502766572 * mass_lower}" />
       <inertia
         ixx="1.493573E-03"
@@ -958,5 +959,5 @@
         rpy="0 0 0" />
       <mass
-        value="${0.0278306854029525 * mass_multi}" />
+        value="${0.0278306854029525 * mass_lower}" />
       <inertia
         ixx="1.48269E-04"
@@ -1014,5 +1015,5 @@
         rpy="0 0 0" />
       <mass
-        value="${0.177450615338578 * mass_multi}" />
+        value="${0.177450615338578 * mass_lower}" />
       <inertia
         ixx="3.75156E-04"
@@ -1070,5 +1071,5 @@
         rpy="0 0 0" />
       <mass
-        value="${0.133904507779755 * mass_multi}" />
+        value="${0.133904507779755 * mass_lower}" />
       <inertia
         ixx="6.95451E-04"
@@ -1127,5 +1128,5 @@
         rpy="0 -1.5708 0" />
       <mass
-        value="${0.00912844677087833 * mass_multi}" />
+        value="${0.00912844677087833 * mass_upper}" />
       <inertia
         ixx="0"
