Commit message: recalculated the inertia

File: dancer_urdf_model/robots/dancer_urdf_model.xacro (robot description, xacro)
@@ -4,6 +4,6 @@
   <xacro:property name="dam" value="0.0"/>
   <xacro:property name="fri" value="10.0"/>
-  <xacro:property name="mass_upper" value="0.4"/>
-  <xacro:property name="mass_lower" value="2.0"/>
+  <xacro:property name="mass_upper" value="1.0"/>
+  <xacro:property name="mass_lower" value="1.0"/>
 <!-- root link -->
   <link
@@ -25,10 +25,10 @@
         value="${0.66907 * mass_upper}" />
       <inertia
-        ixx="0.004463976"
-        ixy="-2.3195E-05"
-        ixz="-2.9057E-05"
-        iyy="0.001971292"
-        iyz="0.000795973"
-        izz="0.004874864" />
+        ixx="0.000757521054"
+        ixy="0"
+        ixz="0"
+        iyy="0.000557000775"
+        iyz="0"
+        izz="0.000913481271" />
     </inertial>
     <visual>
@@ -65,10 +65,10 @@
         value="${0.0560380421735799 * mass_upper}" />
       <inertia
-        ixx="6.80542660516315E-06"
-        ixy="2.52790190769969E-07"
-        ixz="2.16353945279601E-13"
-        iyy="1.50295053154063E-06"
-        iyz="1.49161003758429E-12"
-        izz="8.30837713670273E-06" />
+        ixx="0"
+        ixy="0"
+        ixz="0"
+        iyy="0"
+        iyz="0"
+        izz="0" />
     </inertial>
     <visual>
@@ -121,10 +121,10 @@
         value="${0.067365 * mass_upper}" />
       <inertia
-        ixx="2.0873E-05"
-        ixy="2.2756E-10"
-        ixz="9.0633E-10"
-        iyy="6.1663E-06"
-        iyz="-4.8418E-06"
-        izz="1.4707E-05" />
+        ixx="1.7946036e-05"
+        ixy="0"
+        ixz="0"
+        iyy="1.471574952e-05"
+        iyz="0"
+        izz="1.471574952e-05" />
     </inertial>
     <visual>
@@ -175,12 +175,12 @@
         rpy="0 0 0" />
       <mass
-        value="${0.142976459032186 * mass_upper}" />
-      <inertia
-        ixx="2.49420588469075E-04"
-        ixy="7.32525652321763E-06"
-        ixz="7.10318603096419E-06"
-        iyy="5.00248806790026E-05"
-        iyz="-1.63332458191431E-05"
-        izz="2.60415991235315E-04" />
+        value="${0.14297 * mass_upper}" />
+      <inertia
+        ixx="0.00017824813344"
+        ixy="0"
+        ixz="0"
+        iyy="1.9043604e-05"
+        iyz="0"
+        izz="0.00018358034256" />
     </inertial>
     <visual>
@@ -231,12 +231,12 @@
         rpy="0 0 0" />
       <mass
-        value="${0.021948273112724 * mass_upper}" />
-      <inertia
-        ixx="1.788488E-04"
-        ixy="1.5091E-06"
-        ixz="2.887E-07"
-        iyy="1.97466E-05"
-        iyz="-4.6652E-05"
-        izz="1.653651E-04" />
+        value="${0.02194 * mass_upper}" />
+      <inertia
+        ixx="2.676925728e-05"
+        ixy="0"
+        ixz="0"
+        iyy="4.9680936e-07"
+        iyz="0"
+        izz="2.633089608e-05" />
     </inertial>
     <visual>
@@ -289,10 +289,10 @@
         value="${0.141656759847187 * mass_upper}" />
       <inertia
-        ixx="2.44964545549609E-04"
-        ixy="7.19058779167484E-06"
-        ixz="-7.15162953626525E-06"
-        iyy="4.95100328023302E-05"
-        iyz="1.49143124694347E-05"
-        izz="2.56465619549068E-04" />
+        ixx="0.00017824813344"
+        ixy="0"
+        ixz="0"
+        iyy="1.9043604e-05"
+        iyz="0"
+        izz="0.00018358034256" />
     </inertial>
     <visual>
@@ -345,10 +345,10 @@
         value="${0.021948273112724 * mass_upper}" />
       <inertia
-        ixx="1.442092E-04"
-        ixy="-1.4346E-06"
-        ixz="1.133E-07"
-        iyy="2.13862E-05"
-        iyz="-3.4331E-05"
-        izz="1.307919E-04" />
+        ixx="2.676925728e-05"
+        ixy="0"
+        ixz="0"
+        iyy="4.9680936e-07"
+        iyz="0"
+        izz="2.633089608e-05" />
     </inertial>
     <visual>
@@ -399,12 +399,12 @@
         rpy="0 0 0" />
       <mass
-        value="${0.220741166410594 * mass_upper}" />
-      <inertia
-        ixx="8.47561E-04"
-        ixy="-2.48E-07"
-        ixz="2.243E-06"
-        iyy="1.282726E-03"
-        iyz="1.77836E-03"
-        izz="6.52182E-04" />
+        value="${0.22074 * mass_upper}" />
+      <inertia
+        ixx="4.59415125e-05"
+        ixy="0"
+        ixz="0"
+        iyy="0.00014701284"
+        iyz="0"
+        izz="0.0001341492165" />
     </inertial>
     <visual>
@@ -455,12 +455,12 @@
         rpy="0 0 0" />
       <mass
-        value="${0.0513468076618724 * mass_lower}" />
-      <inertia
-        ixx="3.0932E-05"
-        ixy="5.169E-06"
-        ixz="-2.37E-07"
-        iyy="3.7908E-05"
-        iyz="-9.01E-07"
-        izz="5.787E-05" />
+        value="${0.05134 * mass_lower}" />
+      <inertia
+        ixx="3.419244e-05"
+        ixy="0"
+        ixz="0"
+        iyy="1.3676976e-05"
+        iyz="0"
+        izz="3.419244e-05" />
     </inertial>
     <visual>
@@ -511,12 +511,12 @@
         rpy="0 0 0" />
       <mass
-        value="${0.178226116015845 * mass_lower}" />
-      <inertia
-        ixx="1.44373E-04"
-        ixy="2.00004E-04"
-        ixz="-1.1018E-05"
-        iyy="9.9867E-04"
-        iyz="-4.59E-06"
-        izz="1.074915E-03" />
+        value="${0.17822 * mass_lower}" />
+      <inertia
+        ixx="4.7477808e-05"
+        ixy="0"
+        ixz="0"
+        iyy="0.00011869452"
+        iyz="0"
+        izz="0.00011869452" />
     </inertial>
     <visual>
@@ -567,12 +567,12 @@
         rpy="0 0 0" />
       <mass
-        value="${0.117898503490257 * mass_lower}" />
-      <inertia
-        ixx="1.493574E-03"
-        ixy="-2.86808E-04"
-        ixz="1.94137E-04"
-        iyy="6.08655E-04"
-        iyz="-6.80889E-04"
-        izz="1.149959E-03" />
+        value="${0.11789 * mass_lower}" />
+      <inertia
+        ixx="0.000427905333"
+        ixy="0"
+        ixz="0"
+        iyy="7.0663266e-05"
+        iyz="0"
+        izz="0.000427905333" />
     </inertial>
     <visual>
@@ -623,12 +623,12 @@
         rpy="0 0 0" />
       <mass
-        value="${0.0278306854029525 * mass_lower}" />
-      <inertia
-        ixx="1.48269E-04"
-        ixy="-3.4191E-05"
-        ixz="-1.5824E-05"
-        iyy="5.5445E-05"
-        iyz="5.4765E-05"
-        izz="1.50355E-04" />
+        value="${0.02783 * mass_lower}" />
+      <inertia
+        ixx="0.000101014551"
+        ixy="0"
+        ixz="0"
+        iyy="1.6681302e-05"
+        iyz="0"
+        izz="0.000101014551" />
     </inertial>
     <visual>
@@ -679,12 +679,12 @@
         rpy="0 0 0" />
       <mass
-        value="${0.177450614870689 * mass_lower}" />
-      <inertia
-        ixx="3.75156E-04"
-        ixy="6.1747E-05"
-        ixz="1.24335E-04"
-        iyy="4.65331E-04"
-        iyz="3.8916E-05"
-        izz="2.71139E-04" />
+        value="${0.17745 * mass_lower}" />
+      <inertia
+        ixx="0.0001181817"
+        ixy="0"
+        ixz="0"
+        iyy="0.000147727125"
+        iyz="0"
+        izz="7.6818105e-05" />
     </inertial>
     <visual>
@@ -735,12 +735,12 @@
         rpy="0 0 0" />
       <mass
-        value="${0.13465253780049 * mass_lower}" />
-      <inertia
-        ixx="6.9952E-04"
-        ixy="-3.8103E-05"
-        ixz="3.2233E-05"
-        iyy="5.97429E-04"
-        iyz="-1.8846E-04"
-        izz="3.21756E-04" />
+        value="${0.13465 * mass_lower}" />
+      <inertia
+        ixx="0.00046631988"
+        ixy="0"
+        ixz="0"
+        iyy="0.00060980292"
+        iyz="0"
+        izz="0.0001793538" />
     </inertial>
     <visual>
@@ -793,10 +793,10 @@
         value="${0.0513468076618724 * mass_lower}" />
       <inertia
-        ixx="3.6027E-05"
-        ixy="7.945E-06"
-        ixz="4.126E-06"
-        iyy="4.8251E-05"
-        iyz="2.2027E-06"
-        izz="3.0932E-05" />
+        ixx="3.419244e-05"
+        ixy="0"
+        ixz="0"
+        iyy="1.3676976e-05"
+        iyz="0"
+        izz="3.419244e-05" />
     </inertial>
     <visual>
@@ -849,10 +849,10 @@
         value="${0.178226118022815 * mass_lower}" />
       <inertia
-        ixx="1.44373E-04"
-        ixy="1.48828E-04"
-        ixz="-1.37149E-04"
-        iyy="1.050707E-03"
-        iyz="-3.8299E-05"
-        izz="1.056219E-03" />
+        ixx="4.7477808e-05"
+        ixy="0"
+        ixz="0"
+        iyy="0.00011869452"
+        iyz="0"
+        izz="0.00011869452" />
     </inertial>
     <visual>
@@ -905,10 +905,10 @@
         value="${0.117898502766572 * mass_lower}" />
       <inertia
-        ixx="1.493573E-03"
-        ixy="7.188E-05"
-        ixz="3.94085E-04"
-        iyy="1.596841E-03"
-        iyz="2.56955E-04"
-        izz="2.2449E-04" />
+        ixx="0.000427905333"
+        ixy="0"
+        ixz="0"
+        iyy="7.0663266e-05"
+        iyz="0"
+        izz="0.000427905333" />
     </inertial>
     <visual>
@@ -961,10 +961,10 @@
         value="${0.0278306854029525 * mass_lower}" />
       <inertia
-        ixx="1.48269E-04"
-        ixy="3.7651E-05"
-        ixz="1.9682E-05"
-        iyy="6.588E-05"
-        iyz="5.9917E-05"
-        izz="1.47393E-04" />
+        ixx="0.000101014551"
+        ixy="0"
+        ixz="0"
+        iyy="1.6681302e-05"
+        iyz="0"
+        izz="0.000101014551" />
     </inertial>
     <visual>
@@ -1017,10 +1017,10 @@
         value="${0.177450615338578 * mass_lower}" />
       <inertia
-        ixx="3.75156E-04"
-        ixy="-1.36115E-04"
-        ixz="-6.9757E-05"
-        iyy="3.0154E-04"
-        iyz="4.0854E-05"
-        izz="4.94134E-04" />
+        ixx="0.0001181817"
+        ixy="0"
+        ixz="0"
+        iyy="0.000147727125"
+        iyz="0"
+        izz="7.6818105e-05" />
     </inertial>
     <visual>
@@ -1073,10 +1073,10 @@
         value="${0.133904507779755 * mass_lower}" />
       <inertia
-        ixx="6.95451E-04"
-        ixy="-3.8103E-05"
-        ixz="3.2233E-05"
-        iyy="5.93792E-04"
-        iyz="-1.87682E-04"
-        izz="3.21213E-04" />
+        ixx="0.00046631988"
+        ixy="0"
+        ixz="0"
+        iyy="0.00060980292"
+        iyz="0"
+        izz="0.0001793538" />
     </inertial>
     <visual>
@@ -1193,16 +1193,51 @@
     <mu1>0.2</mu1>
     <mu2>0.2</mu2>
+    <material>Gazebo/Yellow</material>
+    <gravity>true</gravity>
+    <!--<turnGravityoff>false</turnGravityoff>-->
+  </gazebo>
+  <gazebo reference="arm_left">
+    <mu1>0.2</mu1>
+    <mu2>0.2</mu2>
+    <material>Gazebo/Orange</material>
+    <gravity>true</gravity>
+    <!--<turnGravityoff>false</turnGravityoff>-->
+  </gazebo>
+  <gazebo reference="hand_left">
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
Commit message: change fri and mass and mu to lift

File: dancer_urdf_model/robots/dancer_urdf_model.xacro (robot description, xacro)
@@ -3,7 +3,9 @@
   name="dancer_urdf_model" xmlns:xacro="http://www.ros.org/wiki/xacro">
   <xacro:property name="dam" value="0.0"/>
-  <xacro:property name="fri" value="10.0"/>
-  <xacro:property name="mass_upper" value="1.0"/>
-  <xacro:property name="mass_lower" value="1.0"/>
+  <xacro:property name="fri" value="5.0"/>
+  <xacro:property name="mass_upper" value="0.6"/>
+  <xacro:property name="mass_lower" value="2.0"/>
+  <xacro:property name="gazebo_mu1" value="100000"/>
+  <xacro:property name="gazebo_mu2" value="100000"/>
 <!-- root link -->
   <link
@@ -1177,6 +1179,6 @@
 <!-- gazebo -->
   <gazebo reference="body_chest">
-    <mu1>0.2</mu1>
-    <mu2>0.2</mu2>
+    <mu1>${gazebo_mu1}</mu1>
+    <mu2>${gazebo_mu2}</mu2>
     <material>Gazebo/Gray</material>
     <gravity>true</gravity>
@@ -1184,6 +1186,6 @@
   </gazebo>
   <gazebo reference="body_head">
-    <mu1>0.2</mu1>
-    <mu2>0.2</mu2>
+    <mu1>${gazebo_mu1}</mu1>
+    <mu2>${gazebo_mu2}</mu2>
     <material>Gazebo/Green</material>
     <gravity>true</gravity>
@@ -1191,6 +1193,6 @@
   </gazebo>
   <gazebo reference="body_head2">
-    <mu1>0.2</mu1>
-    <mu2>0.2</mu2>
+    <mu1>${gazebo_mu1}</mu1>
+    <mu2>${gazebo_mu2}</mu2>
     <material>Gazebo/Yellow</material>
     <gravity>true</gravity>
@@ -1198,6 +1200,6 @@
   </gazebo>
   <gazebo reference="arm_left">
-    <mu1>0.2</mu1>
-    <mu2>0.2</mu2>
+    <mu1>${gazebo_mu1}</mu1>
+    <mu2>${gazebo_mu2}</mu2>
     <material>Gazebo/Orange</material>
     <gravity>true</gravity>
@@ -1205,6 +1207,6 @@
   </gazebo>
   <gazebo reference="hand_left">
-    <mu1>0.2</mu1>
-    <mu2>0.2</mu2>
+    <mu1>${gazebo_mu1}</mu1>
+    <mu2>${gazebo_mu2}</mu2>
     <material>Gazebo/Yellow</material>
     <gravity>true</gravity>
@@ -1212,6 +1214,6 @@
   </gazebo>
   <gazebo reference="arm_right">
-    <mu1>0.2</mu1>
-    <mu2>0.2</mu2>
+    <mu1>${gazebo_mu1}</mu1>
+    <mu2>${gazebo_mu2}</mu2>
     <material>Gazebo/Black</material>
     <gravity>true</gravity>
@@ -1219,6 +1221,6 @@
   </gazebo>
   <gazebo reference="hand_right">
-    <mu1>0.2</mu1>
-    <mu2>0.2</mu2>
+    <mu1>${gazebo_mu1}</mu1>
+    <mu2>${gazebo_mu2}</mu2>
     <material>Gazebo/Black</material>
     <gravity>true</gravity>
@@ -1226,6 +1228,6 @@
   </gazebo>
   <gazebo reference="body_hip">
-    <mu1>0.2</mu1>
-    <mu2>0.2</mu2>
+    <mu1>${gazebo_mu1}</mu1>
+    <mu2>${gazebo_mu2}</mu2>
     <material>Gazebo/Green</material>
     <gravity>true</gravity>
@@ -1233,6 +1235,6 @@
   </gazebo>
   <gazebo reference="body_hip_left">
-    <mu1>0.2</mu1>
-    <mu2>0.2</mu2>
+    <mu1>${gazebo_mu1}</mu1>
+    <mu2>${gazebo_mu2}</mu2>
     <material>Gazebo/Yellow</material>
     <gravity>true</gravity>
@@ -1240,6 +1242,6 @@
   </gazebo>
   <gazebo reference="body_hip2_left">
-    <mu1>0.2</mu1>
-    <mu2>0.2</mu2>
+    <mu1>${gazebo_mu1}</mu1>
+    <mu2>${gazebo_mu2}</mu2>
     <material>Gazebo/Orange</material>
     <gravity>true</gravity>
@@ -1247,6 +1249,6 @@
   </gazebo>
   <gazebo reference="leg_left">
-    <mu1>0.2</mu1>
-    <mu2>0.2</mu2>
+    <mu1>${gazebo_mu1}</mu1>
+    <mu2>${gazebo_mu2}</mu2>
     <material>Gazebo/Yellow</material>
     <gravity>true</gravity>
@@ -1254,6 +1256,6 @@
   </gazebo>
   <gazebo reference="leg2_left">
-    <mu1>0.2</mu1>
-    <mu2>0.2</mu2>
+    <mu1>${gazebo_mu1}</mu1>
+    <mu2>${gazebo_mu2}</mu2>
     <material>Gazebo/Orange</material>
     <gravity>true</gravity>
@@ -1261,6 +1263,6 @@
   </gazebo>
   <gazebo reference="leg3_left">
-    <mu1>0.2</mu1>
-    <mu2>0.2</mu2>
+    <mu1>${gazebo_mu1}</mu1>
+    <mu2>${gazebo_mu2}</mu2>
     <material>Gazebo/Yellow</material>
     <gravity>true</gravity>
@@ -1268,6 +1270,6 @@
   </gazebo>
   <gazebo reference="leg4_left">
-    <mu1>0.2</mu1>
-    <mu2>0.2</mu2>
+    <mu1>${gazebo_mu1}</mu1>
+    <mu2>${gazebo_mu2}</mu2>
     <material>Gazebo/Orange</material>
     <gravity>true</gravity>
@@ -1275,6 +1277,6 @@
   </gazebo>
   <gazebo reference="body_hip_right">
-    <mu1>0.2</mu1>
-    <mu2>0.2</mu2>
+    <mu1>${gazebo_mu1}</mu1>
+    <mu2>${gazebo_mu2}</mu2>
     <material>Gazebo/Yellow</material>
     <gravity>true</gravity>
@@ -1282,6 +1284,6 @@
   </gazebo>
   <gazebo reference="body_hip2_right">
-    <mu1>0.2</mu1>
-    <mu2>0.2</mu2>
+    <mu1>${gazebo_mu1}</mu1>
+    <mu2>${gazebo_mu2}</mu2>
     <material>Gazebo/Orange</material>
     <gravity>true</gravity>
@@ -1289,6 +1291,6 @@
   </gazebo>
   <gazebo reference="leg_right">
-    <mu1>0.2</mu1>
-    <mu2>0.2</mu2>
+    <mu1>${gazebo_mu1}</mu1>
+    <mu2>${gazebo_mu2}</mu2>
     <material>Gazebo/Black</material>
     <gravity>true</gravity>
@@ -1296,6 +1298,6 @@
   </gazebo>
   <gazebo reference="leg2_right">
-    <mu1>0.2</mu1>
-    <mu2>0.2</mu2>
+    <mu1>${gazebo_mu1}</mu1>
+    <mu2>${gazebo_mu2}</mu2>
     <material>Gazebo/Black</material>
     <gravity>true</gravity>
@@ -1303,6 +1305,6 @@
   </gazebo>
   <gazebo reference="leg3_right">
-    <mu1>0.2</mu1>
-    <mu2>0.2</mu2>
+    <mu1>${gazebo_mu1}</mu1>
+    <mu2>${gazebo_mu2}</mu2>
      <material>Gazebo/Black</material>
     <gravity>true</gravity>
@@ -1310,6 +1312,6 @@
   </gazebo>
   <gazebo reference="leg4_right">
-    <mu1>0.2</mu1>
-    <mu2>0.2</mu2>
+    <mu1>${gazebo_mu1}</mu1>
+    <mu2>${gazebo_mu2}</mu2>
     <material>Gazebo/Black</material>
     <gravity>true</gravity>
@@ -1317,6 +1319,6 @@
   </gazebo>
   <gazebo reference="body_camera">
-    <mu1>0.2</mu1>
-    <mu2>0.2</mu2>
+    <mu1>${gazebo_mu1}</mu1>
+    <mu2>${gazebo_mu2}</mu2>
     <material>Gazebo/Red</material>
     <sensor type="camera" name="camera1">

Commit message: use txt data to init state

File: dancer_urdf_model/robots/dancer_urdf_model.xacro (robot description, xacro)
@@ -3,7 +3,7 @@
   name="dancer_urdf_model" xmlns:xacro="http://www.ros.org/wiki/xacro">
   <xacro:property name="dam" value="0.0"/>
-  <xacro:property name="fri" value="5.0"/>
-  <xacro:property name="mass_upper" value="0.6"/>
-  <xacro:property name="mass_lower" value="2.0"/>
+  <xacro:property name="fri" value="10.0"/>
+  <xacro:property name="mass_upper" value="1.0"/>
+  <xacro:property name="mass_lower" value="1.0"/>
   <xacro:property name="gazebo_mu1" value="100000"/>
   <xacro:property name="gazebo_mu2" value="100000"/>

Commit message: 站起来了

File: dancer_urdf_model/robots/dancer_urdf_model.xacro (robot description, xacro)
@@ -2,8 +2,12 @@
 <robot
   name="dancer_urdf_model" xmlns:xacro="http://www.ros.org/wiki/xacro">
+  <!--关节阻尼与摩擦力-->
   <xacro:property name="dam" value="0.0"/>
-  <xacro:property name="fri" value="10.0"/>
-  <xacro:property name="mass_upper" value="1.0"/>
-  <xacro:property name="mass_lower" value="1.0"/>
+  <xacro:property name="fri" value="20.0"/>
+  <!--上半身与下半身质量系数-->
+  <xacro:property name="mass_upper" value="1.0"/><!--head,arm,hand,hip-->
+  <xacro:property name="mass_middle" value="3.0"/><!--hipleft,hipleft2,leg1-->
+  <xacro:property name="mass_lower" value="10.0"/><!--leg2,leg3,leg4-->
+  <!--gazebo摩擦力-->
   <xacro:property name="gazebo_mu1" value="100000"/>
   <xacro:property name="gazebo_mu2" value="100000"/>
@@ -457,5 +461,5 @@
         rpy="0 0 0" />
       <mass
-        value="${0.05134 * mass_lower}" />
+        value="${0.05134 * mass_middle}" />
       <inertia
         ixx="3.419244e-05"
@@ -513,5 +517,5 @@
         rpy="0 0 0" />
       <mass
-        value="${0.17822 * mass_lower}" />
+        value="${0.17822 * mass_middle}" />
       <inertia
         ixx="4.7477808e-05"
@@ -569,5 +573,5 @@
         rpy="0 0 0" />
       <mass
-        value="${0.11789 * mass_lower}" />
+        value="${0.11789 * mass_middle}" />
       <inertia
         ixx="0.000427905333"
@@ -793,5 +797,5 @@
         rpy="0 0 0" />
       <mass
-        value="${0.0513468076618724 * mass_lower}" />
+        value="${0.0513468076618724 * mass_middle}" />
       <inertia
         ixx="3.419244e-05"
@@ -849,5 +853,5 @@
         rpy="0 0 0" />
       <mass
-        value="${0.178226118022815 * mass_lower}" />
+        value="${0.178226118022815 * mass_middle}" />
       <inertia
         ixx="4.7477808e-05"
@@ -905,5 +909,5 @@
         rpy="0 0 0" />
       <mass
-        value="${0.117898502766572 * mass_lower}" />
+        value="${0.117898502766572 * mass_middle}" />
       <inertia
         ixx="0.000427905333"

Commit message: 调节了PID和关节参数

File: dancer_urdf_model/robots/dancer_urdf_model.xacro (robot description, xacro)
@@ -4,9 +4,12 @@
   <!--关节阻尼与摩擦力-->
   <xacro:property name="dam" value="0.0"/>
-  <xacro:property name="fri" value="20.0"/>
+  <xacro:property name="fri" value="1.0"/>
+  <!--关节转动限制-->
+  <xacro:property name="lim_effort" value="10000.0"/>
+  <xacro:property name="lim_vel" value="10.0"/>
   <!--上半身与下半身质量系数-->
   <xacro:property name="mass_upper" value="1.0"/><!--head,arm,hand,hip-->
-  <xacro:property name="mass_middle" value="3.0"/><!--hipleft,hipleft2,leg1-->
-  <xacro:property name="mass_lower" value="10.0"/><!--leg2,leg3,leg4-->
+  <xacro:property name="mass_middle" value="4.0"/><!--hipleft,hipleft2,leg1-->
+  <xacro:property name="mass_lower" value="9.0"/><!--leg2,leg3,leg4-->
   <!--gazebo摩擦力-->
   <xacro:property name="gazebo_mu1" value="100000"/>
@@ -117,4 +120,7 @@
       damping="${dam}"
       friction="${fri}" />
+    <limit
+      effort="${lim_effort}"
+      velocity="${lim_vel}" />
   </joint>
   <link
@@ -173,4 +179,7 @@
       damping="${dam}"
       friction="${fri}" />
+    <limit
+      effort="${lim_effort}"
+      velocity="${lim_vel}" />
   </joint>
   <link
@@ -229,4 +238,7 @@
       damping="${dam}"
       friction="${fri}" />
+    <limit
+      effort="${lim_effort}"
+      velocity="${lim_vel}" />
   </joint>
   <link
@@ -285,4 +297,7 @@
       damping="${dam}"
       friction="${fri}" />
+    <limit
+      effort="${lim_effort}"
+      velocity="${lim_vel}" />
   </joint>
   <link
@@ -341,4 +356,7 @@
       damping="${dam}"
       friction="${fri}" />
+    <limit
+      effort="${lim_effort}"
+      velocity="${lim_vel}" />
   </joint>
   <link
@@ -397,4 +415,7 @@
       damping="${dam}"
       friction="${fri}" />
+    <limit
+      effort="${lim_effort}"
+      velocity="${lim_vel}" />
   </joint>
   <link
@@ -453,4 +474,7 @@
       damping="${dam}"
       friction="${fri}" />
+    <limit
+      effort="${lim_effort}"
+      velocity="${lim_vel}" />
   </joint>
   <link
@@ -509,4 +533,7 @@
       damping="${dam}"
       friction="${fri}" />
+    <limit
+      effort="${lim_effort}"
+      velocity="${lim_vel}" />
   </joint>
   <link
@@ -565,4 +592,7 @@
       damping="${dam}"
       friction="${fri}" />
+    <limit
+      effort="${lim_effort}"
+      velocity="${lim_vel}" />
   </joint>
   <link
@@ -621,4 +651,7 @@
       damping="${dam}"
       friction="${fri}" />
+    <limit
+      effort="${lim_effort}"
+      velocity="${lim_vel}" />
   </joint>
   <link
@@ -677,4 +710,7 @@
       damping="${dam}"
       friction="${fri}" />
+    <limit
+      effort="${lim_effort}"
+      velocity="${lim_vel}" />
   </joint>
   <link
@@ -733,4 +769,7 @@
       damping="${dam}"
       friction="${fri}" />
+    <limit
+      effort="${lim_effort}"
+      velocity="${lim_vel}" />
   </joint>
   <link
@@ -789,4 +828,7 @@
       damping="${dam}"
       friction="${fri}" />
+    <limit
+      effort="${lim_effort}"
+      velocity="${lim_vel}" />
   </joint>
   <link
@@ -845,4 +887,7 @@
       damping="${dam}"
       friction="${fri}" />
+    <limit
+      effort="${lim_effort}"
+      velocity="${lim_vel}" />
   </joint>
   <link
@@ -901,4 +946,7 @@
       damping="${dam}"
       friction="${fri}" />
+    <limit
+      effort="${lim_effort}"
+      velocity="${lim_vel}" />
   </joint>
   <link
@@ -957,4 +1005,7 @@
       damping="${dam}"
       friction="${fri}" />
+    <limit
+      effort="${lim_effort}"
+      velocity="${lim_vel}" />
   </joint>
   <link
@@ -1013,4 +1064,7 @@
       damping="${dam}"
       friction="${fri}" />
+    <limit
+      effort="${lim_effort}"
+      velocity="${lim_vel}" />
   </joint>
   <link
@@ -1069,4 +1123,7 @@
       damping="${dam}"
       friction="${fri}" />
+    <limit
+      effort="${lim_effort}"
+      velocity="${lim_vel}" />
   </joint>
   <link
@@ -1125,4 +1182,7 @@
       damping="${dam}"
       friction="${fri}" />
+    <limit
+      effort="${lim_effort}"
+      velocity="${lim_vel}" />
   </joint>
 <!-- camera -->
