Commit message: 拆分质量系数和ＰＩＤ的ｐ为身体四个部分，分别整定

File: dancer_urdf_model/robots/dancer_urdf_model.xacro (robot description, xacro)
@@ -9,7 +9,8 @@
   <xacro:property name="lim_vel" value="10.0"/>
   <!--上半身与下半身质量系数-->
-  <xacro:property name="mass_upper" value="1.0"/><!--head,arm,hand,hip-->
+  <xacro:property name="mass_upper" value="1.0"/><!--head,hip-->
+  <xacro:property name="mass_hands" value="1.0"/><!--arm,hand-->
   <xacro:property name="mass_middle" value="4.0"/><!--hipleft,hipleft2,leg1-->
-  <xacro:property name="mass_lower" value="9.0"/><!--leg2,leg3,leg4-->
+  <xacro:property name="mass_lower" value="8.0"/><!--leg2,leg3,leg4-->
   <!--gazebo摩擦力-->
   <xacro:property name="gazebo_mu1" value="100000"/>
@@ -190,5 +191,5 @@
         rpy="0 0 0" />
       <mass
-        value="${0.14297 * mass_upper}" />
+        value="${0.14297 * mass_hands}" />
       <inertia
         ixx="0.00017824813344"
@@ -249,5 +250,5 @@
         rpy="0 0 0" />
       <mass
-        value="${0.02194 * mass_upper}" />
+        value="${0.02194 * mass_hands}" />
       <inertia
         ixx="2.676925728e-05"
@@ -308,5 +309,5 @@
         rpy="0 0 0" />
       <mass
-        value="${0.141656759847187 * mass_upper}" />
+        value="${0.141656759847187 * mass_hands}" />
       <inertia
         ixx="0.00017824813344"
@@ -367,5 +368,5 @@
         rpy="0 0 0" />
       <mass
-        value="${0.021948273112724 * mass_upper}" />
+        value="${0.021948273112724 * mass_hands}" />
       <inertia
         ixx="2.676925728e-05"

Commit message: 修正了全身关节初始值和转轴方位

File: dancer_urdf_model/robots/dancer_urdf_model.xacro (robot description, xacro)
@@ -10,5 +10,5 @@
   <!--上半身与下半身质量系数-->
   <xacro:property name="mass_upper" value="1.0"/><!--head,hip-->
-  <xacro:property name="mass_hands" value="1.0"/><!--arm,hand-->
+  <xacro:property name="mass_hands" value="2.0"/><!--arm,hand-->
   <xacro:property name="mass_middle" value="4.0"/><!--hipleft,hipleft2,leg1-->
   <xacro:property name="mass_lower" value="8.0"/><!--leg2,leg3,leg4-->
@@ -524,5 +524,5 @@
     <origin
       xyz="0.045 -0.0122 0.065"
-      rpy="1.5608 0 -1.5708" /><!--rpy="1.5708 0 -1.5708" put 0.01 into r-->
+      rpy="1.6008 0 -1.5708" /><!--rpy="1.5708 0 -1.5708" put 0.03 into r-->
     <parent
       link="body_hip" />
@@ -819,9 +819,9 @@
     <origin
       xyz="-0.0241 -0.0065502 0.035907"
-      rpy="0 0.3368 0.41369" /><!--rpy="-2.9765 -0.0732 0.41369" put 0.41 into p-->
-    <parent
-      link="leg3_left" />
-    <child
-      link="leg4_left" />
+      rpy="-2.9765 -0.0132 0.11369" /><!--rpy="-2.9765 -0.0732 0.41369" put 0.41 into p-->
+    <parent
+      link="leg3_left" /><!-- and put -0.35 into p-->
+    <child
+      link="leg4_left" /><!-- and put -0.30 into y-->
     <axis
       xyz="0 0 1" />
@@ -937,5 +937,5 @@
     <origin
       xyz="0.031042 0.015283 0.0465"
-      rpy="2.309 0 0.4575" /><!--rpy="1.479 0 0.4575" put -0.83 into r-->
+      rpy="2.229 0 0.4575" /><!--rpy="1.479 0 0.4575" put -0.83 into r and put -0.08 into r-->
     <parent
       link="body_hip_right" />
@@ -1055,7 +1055,7 @@
     <origin
       xyz="-0.0016 -0.020351 -0.11826"
-      rpy="0.79 0 0" /><!--rpy="0 0 0" put 0.79 into r-->
-    <parent
-      link="leg_right" />
+      rpy="0.94 0 0" /><!--rpy="0 0 0" put 0.79 into r-->
+    <parent
+      link="leg_right" /><!-- and put 0.15 into r-->
     <child
       link="leg2_right" />
@@ -1172,12 +1172,12 @@
     type="continuous">
     <origin
-      xyz="-0.0265 0 0.0061902"
-      rpy="1.883 0.0941 2.8787" /><!--rpy="1.883 -0.9859 2.8787" put -1.08 into p--><!--xyz="-0.0265 -0.035971 0.0061902"-->
-    <parent
-      link="leg3_right" />
-    <child
-      link="leg4_right" />
-    <axis
-      xyz="0 0 1" />
+      xyz="-0.0265 -0.035971 0.0061902"
+      rpy="1.753 -0.1059 3.1487" /><!--rpy="1.883 -0.9859 2.8787" put -1.08 into p-->
+    <parent
+      link="leg3_right" /><!-- and put 0.27 into y-->
+    <child
+      link="leg4_right" /><!-- and put -0.13 into r-->
+    <axis
+      xyz="0 0 1" /><!-- and put -0.20 into p-->
     <dynamics
       damping="${dam}"

Commit message: 勉强能走但抬腿无力，PID还需调节

File: dancer_urdf_model/robots/dancer_urdf_model.xacro (robot description, xacro)
@@ -12,5 +12,5 @@
   <xacro:property name="mass_hands" value="2.0"/><!--arm,hand-->
   <xacro:property name="mass_middle" value="4.0"/><!--hipleft,hipleft2,leg1-->
-  <xacro:property name="mass_lower" value="8.0"/><!--leg2,leg3,leg4-->
+  <xacro:property name="mass_lower" value="10.0"/><!--leg2,leg3,leg4-->
   <!--gazebo摩擦力-->
   <xacro:property name="gazebo_mu1" value="100000"/>
@@ -73,5 +73,5 @@
         rpy="0 0 0" />
       <mass
-        value="${0.0560380421735799 * mass_upper}" />
+        value="${0.05603 * mass_upper}" />
       <inertia
         ixx="0"
@@ -132,5 +132,5 @@
         rpy="0 0 0" />
       <mass
-        value="${0.067365 * mass_upper}" />
+        value="${0.06736 * mass_upper}" />
       <inertia
         ixx="1.7946036e-05"
@@ -309,5 +309,5 @@
         rpy="0 0 0" />
       <mass
-        value="${0.141656759847187 * mass_hands}" />
+        value="${0.14165 * mass_hands}" />
       <inertia
         ixx="0.00017824813344"
@@ -368,5 +368,5 @@
         rpy="0 0 0" />
       <mass
-        value="${0.021948273112724 * mass_hands}" />
+        value="${0.02194 * mass_hands}" />
       <inertia
         ixx="2.676925728e-05"
@@ -760,7 +760,7 @@
     <origin
       xyz="0.0006 0.11852 0.05341"
-      rpy="0.19 0 0" /><!--rpy="0 0 0" put -0.19 into r-->
-    <parent
-      link="leg2_left" />
+      rpy="0.36 0 0" /><!--rpy="0 0 0" put -0.19 * -1 into r-->
+    <parent
+      link="leg2_left" /><!-- put 0.17 into r to prevent falling-->
     <child
       link="leg3_left" />
@@ -840,5 +840,5 @@
         rpy="0 0 0" />
       <mass
-        value="${0.0513468076618724 * mass_middle}" />
+        value="${0.05134 * mass_middle}" />
       <inertia
         ixx="3.419244e-05"
@@ -899,5 +899,5 @@
         rpy="0 0 0" />
       <mass
-        value="${0.178226118022815 * mass_middle}" />
+        value="${0.17822 * mass_middle}" />
       <inertia
         ixx="4.7477808e-05"
@@ -937,7 +937,7 @@
     <origin
       xyz="0.031042 0.015283 0.0465"
-      rpy="2.229 0 0.4575" /><!--rpy="1.479 0 0.4575" put -0.83 into r and put -0.08 into r-->
-    <parent
-      link="body_hip_right" />
+      rpy="2.229 0 0.4575" /><!--rpy="1.479 0 0.4575" put -0.83 * -1 into r-->
+    <parent
+      link="body_hip_right" /><!-- and put -0.08 into r-->
     <child
       link="body_hip2_right" />
@@ -958,5 +958,5 @@
         rpy="0 0 0" />
       <mass
-        value="${0.117898502766572 * mass_middle}" />
+        value="${0.11789 * mass_middle}" />
       <inertia
         ixx="0.000427905333"
@@ -1017,5 +1017,5 @@
         rpy="0 0 0" />
       <mass
-        value="${0.0278306854029525 * mass_lower}" />
+        value="${0.02783 * mass_lower}" />
       <inertia
         ixx="0.000101014551"
@@ -1076,5 +1076,5 @@
         rpy="0 0 0" />
       <mass
-        value="${0.177450615338578 * mass_lower}" />
+        value="${0.17745 * mass_lower}" />
       <inertia
         ixx="0.0001181817"
@@ -1114,7 +1114,7 @@
     <origin
       xyz="0 -0.1146 -0.061382"
-      rpy="-0.83 0 0" /><!--rpy="0 0 0" put -0.83 into r-->
-    <parent
-      link="leg2_right" />
+      rpy="-0.96 0 0" /><!--rpy="0 0 0" put -0.83 into r-->
+    <parent
+      link="leg2_right" /><!-- put -0.17 into r to prevent falling-->
     <child
       link="leg3_right" />
@@ -1135,5 +1135,5 @@
         rpy="0 0 0" />
       <mass
-        value="${0.133904507779755 * mass_lower}" />
+        value="${0.13390 * mass_lower}" />
       <inertia
         ixx="0.00046631988"
@@ -1195,5 +1195,5 @@
         rpy="0 -1.5708 0" />
       <mass
-        value="${0.00912844677087833 * mass_upper}" />
+        value="${0.00912 * mass_upper}" />
       <inertia
         ixx="0"
@@ -1390,5 +1390,5 @@
       <always_on>true</always_on>
       <!--<updateRate>30.0</updateRate>-->
-      <visualize>true</visualize>
+      <visualize>false</visualize>
       <camera name="head">
         <horizontal_fov>1.3962634</horizontal_fov>

Commit message: 调节ＰＩＤ减小震荡勉强能走

File: dancer_urdf_model/robots/dancer_urdf_model.xacro (robot description, xacro)
@@ -6,5 +6,5 @@
   <xacro:property name="fri" value="1.0"/>
   <!--关节转动限制-->
-  <xacro:property name="lim_effort" value="10000.0"/>
+  <xacro:property name="lim_effort" value="1000000.0"/>
   <xacro:property name="lim_vel" value="10.0"/>
   <!--上半身与下半身质量系数-->

Commit message: 调整关节转速与脚底板

File: dancer_urdf_model/robots/dancer_urdf_model.xacro (robot description, xacro)
@@ -7,5 +7,5 @@
   <!--关节转动限制-->
   <xacro:property name="lim_effort" value="1000000.0"/>
-  <xacro:property name="lim_vel" value="10.0"/>
+  <xacro:property name="lim_vel" value="1.0"/>
   <!--上半身与下半身质量系数-->
   <xacro:property name="mass_upper" value="1.0"/><!--head,hip-->
@@ -760,7 +760,7 @@
     <origin
       xyz="0.0006 0.11852 0.05341"
-      rpy="0.36 0 0" /><!--rpy="0 0 0" put -0.19 * -1 into r-->
-    <parent
-      link="leg2_left" /><!-- put 0.17 into r to prevent falling-->
+      rpy="0.41 0 0" /><!--rpy="0 0 0" put -0.19 * -1 into r-->
+    <parent
+      link="leg2_left" /><!-- put 0.22 into r to prevent falling-->
     <child
       link="leg3_left" />
@@ -1114,7 +1114,7 @@
     <origin
       xyz="0 -0.1146 -0.061382"
-      rpy="-0.96 0 0" /><!--rpy="0 0 0" put -0.83 into r-->
-    <parent
-      link="leg2_right" /><!-- put -0.17 into r to prevent falling-->
+      rpy="-1.05 0 0" /><!--rpy="0 0 0" put -0.83 into r-->
+    <parent
+      link="leg2_right" /><!-- put -0.22 into r to prevent falling-->
     <child
       link="leg3_right" />

Commit message: 修正上半身转动惯量与转速限制

File: dancer_urdf_model/robots/dancer_urdf_model.xacro (robot description, xacro)
@@ -6,5 +6,5 @@
   <xacro:property name="fri" value="1.0"/>
   <!--关节转动限制-->
-  <xacro:property name="lim_effort" value="1000000.0"/>
+  <xacro:property name="lim_effort" value="10000000.0"/>
   <xacro:property name="lim_vel" value="1.0"/>
   <!--上半身与下半身质量系数-->
@@ -14,6 +14,6 @@
   <xacro:property name="mass_lower" value="10.0"/><!--leg2,leg3,leg4-->
   <!--gazebo摩擦力-->
-  <xacro:property name="gazebo_mu1" value="100000"/>
-  <xacro:property name="gazebo_mu2" value="100000"/>
+  <xacro:property name="gazebo_mu1" value="0.1"/>
+  <xacro:property name="gazebo_mu2" value="0.1"/>
 <!-- root link -->
   <link
@@ -35,10 +35,10 @@
         value="${0.66907 * mass_upper}" />
       <inertia
-        ixx="${0.000757521054 * sqrt(mass_upper)}"
-        ixy="0"
-        ixz="0"
-        iyy="${0.000557000775 * sqrt(mass_upper)}"
-        iyz="0"
-        izz="${0.000913481271 * sqrt(mass_upper)}" />
+        ixx="${0.003030084216 * sqrt(mass_upper)}"
+        ixy="0"
+        ixz="0"
+        iyy="${0.0022280031 * sqrt(mass_upper)}"
+        iyz="0"
+        izz="${0.003653925084 * sqrt(mass_upper)}" />
     </inertial>
     <visual>
@@ -783,10 +783,10 @@
         value="${0.13465 * mass_lower}" />
       <inertia
-        ixx="${0.00046631988 * sqrt(mass_lower)}"
-        ixy="0"
-        ixz="0"
-        iyy="${0.00060980292 * sqrt(mass_lower)}"
-        iyz="0"
-        izz="${0.0001793538 * sqrt(mass_lower)}" />
+        ixx="${0.000919188225 * sqrt(mass_lower)}"
+        ixy="0"
+        ixz="0"
+        iyy="${0.00132721812 * sqrt(mass_lower)}"
+        iyz="0"
+        izz="${0.000488739105 * sqrt(mass_lower)}" />
     </inertial>
     <visual>
@@ -1137,10 +1137,10 @@
         value="${0.13390 * mass_lower}" />
       <inertia
-        ixx="${0.00046631988 * sqrt(mass_lower)}"
-        ixy="0"
-        ixz="0"
-        iyy="${0.00060980292 * sqrt(mass_lower)}"
-        iyz="0"
-        izz="${0.0001793538 * sqrt(mass_lower)}" />
+        ixx="${0.000919188225 * sqrt(mass_lower)}"
+        ixy="0"
+        ixz="0"
+        iyy="${0.00132721812 * sqrt(mass_lower)}"
+        iyz="0"
+        izz="${0.000488739105 * sqrt(mass_lower)}" />
     </inertial>
     <visual>

Commit message: 双腿初始并拢，修正头部小臂转动惯量

File: dancer_urdf_model/robots/dancer_urdf_model.xacro (robot description, xacro)
@@ -4,5 +4,5 @@
   <!--关节阻尼与摩擦力-->
   <xacro:property name="dam" value="0.0"/>
-  <xacro:property name="fri" value="1.0"/>
+  <xacro:property name="fri" value="0.0"/>
   <!--关节转动限制-->
   <xacro:property name="lim_effort" value="10000000.0"/>
@@ -14,6 +14,6 @@
   <xacro:property name="mass_lower" value="10.0"/><!--leg2,leg3,leg4-->
   <!--gazebo摩擦力-->
-  <xacro:property name="gazebo_mu1" value="0.1"/>
-  <xacro:property name="gazebo_mu2" value="0.1"/>
+  <xacro:property name="gazebo_mu1" value="0.8"/>
+  <xacro:property name="gazebo_mu2" value="0.8"/>
 <!-- root link -->
   <link
@@ -35,10 +35,10 @@
         value="${0.66907 * mass_upper}" />
       <inertia
-        ixx="${0.003030084216 * sqrt(mass_upper)}"
-        ixy="0"
-        ixz="0"
-        iyy="${0.0022280031 * sqrt(mass_upper)}"
-        iyz="0"
-        izz="${0.003653925084 * sqrt(mass_upper)}" />
+        ixx="${0.001448202015 * sqrt(mass_upper)}"
+        ixy="0"
+        ixz="0"
+        iyy="${0.000913481271 * sqrt(mass_upper)}"
+        iyz="0"
+        izz="${0.001648722294 * sqrt(mass_upper)}" />
     </inertial>
     <visual>
@@ -75,10 +75,10 @@
         value="${0.05603 * mass_upper}" />
       <inertia
-        ixx="0"
-        ixy="0"
-        ixz="0"
-        iyy="0"
-        iyz="0"
-        izz="0" />
+        ixx="${1.7946036e-05 * sqrt(mass_upper)}"
+        ixy="0"
+        ixz="0"
+        iyy="${1.471574952e-05 * sqrt(mass_upper)}"
+        iyz="0"
+        izz="${1.471574952e-05 * sqrt(mass_upper)}" />
     </inertial>
     <visual>
@@ -134,10 +134,10 @@
         value="${0.06736 * mass_upper}" />
       <inertia
-        ixx="${1.7946036e-05 * sqrt(mass_upper)}"
-        ixy="0"
-        ixz="0"
-        iyy="${1.471574952e-05 * sqrt(mass_upper)}"
-        iyz="0"
-        izz="${1.471574952e-05 * sqrt(mass_upper)}" />
+        ixx="${2.4255387e-05 * mass_upper}"
+        ixy="0"
+        ixz="0"
+        iyy="${3.3584382e-05 * mass_upper}"
+        iyz="0"
+        izz="${2.4255387e-05 * mass_upper}" />
     </inertial>
     <visual>
@@ -193,10 +193,10 @@
         value="${0.14297 * mass_hands}" />
       <inertia
-        ixx="${0.00017824813344 * sqrt(mass_hands)}"
-        ixy="0"
-        ixz="0"
-        iyy="${1.9043604e-05 * sqrt(mass_hands)}"
-        iyz="0"
-        izz="${0.00018358034256 * sqrt(mass_hands)}" />
+        ixx="${0.000347545773 * sqrt(mass_hands)}"
+        ixy="0"
+        ixz="0"
+        iyy="${8.5696218e-05 * sqrt(mass_hands)}"
+        iyz="0"
+        izz="${0.000347545773 * sqrt(mass_hands)}" />
     </inertial>
     <visual>
@@ -252,10 +252,10 @@
         value="${0.02194 * mass_hands}" />
       <inertia
-        ixx="${2.676925728e-05 * sqrt(mass_hands)}"
-        ixy="0"
-        ixz="0"
-        iyy="${4.9680936e-07 * sqrt(mass_hands)}"
-        iyz="0"
-        izz="${2.633089608e-05 * sqrt(mass_hands)}" />
+        ixx="${7.5982608e-05 * sqrt(mass_hands)}"
+        ixy="0"
+        ixz="0"
+        iyy="${3.1050585e-06 * sqrt(mass_hands)}"
+        iyz="0"
+        izz="${7.32428505e-05 * sqrt(mass_hands)}" />
     </inertial>
     <visual>
@@ -311,10 +311,10 @@
         value="${0.14165 * mass_hands}" />
       <inertia
-        ixx="${0.00017824813344 * sqrt(mass_hands)}"
-        ixy="0"
-        ixz="0"
-        iyy="${1.9043604e-05 * sqrt(mass_hands)}"
-        iyz="0"
-        izz="${0.00018358034256 * sqrt(mass_hands)}" />
+        ixx="${0.000347545773 * sqrt(mass_hands)}"
+        ixy="0"
+        ixz="0"
+        iyy="${8.5696218e-05 * sqrt(mass_hands)}"
+        iyz="0"
+        izz="${0.000347545773 * sqrt(mass_hands)}" />
     </inertial>
     <visual>
@@ -370,10 +370,10 @@
         value="${0.02194 * mass_hands}" />
       <inertia
-        ixx="${2.676925728e-05 * sqrt(mass_hands)}"
-        ixy="0"
-        ixz="0"
-        iyy="${4.9680936e-07 * sqrt(mass_hands)}"
-        iyz="0"
-        izz="${2.633089608e-05 * sqrt(mass_hands)}" />
+        ixx="${7.5982608e-05 * sqrt(mass_hands)}"
+        ixy="0"
+        ixz="0"
+        iyy="${3.1050585e-06 * sqrt(mass_hands)}"
+        iyz="0"
+        izz="${7.32428505e-05 * sqrt(mass_hands)}" />
     </inertial>
     <visual>
@@ -583,7 +583,7 @@
     <origin
       xyz="0.0493 0.033966 -0.0015267"
-      rpy="3.2898 0.044917 1.5708" /><!--rpy="3.0498 0.044917 1.5708" put -0.14 into -r-->
-    <parent
-      link="body_hip_left" />
+      rpy="3.1698 0.044917 1.5708" /><!--rpy="3.0498 0.044917 1.5708" put -0.14 into -r-->
+    <parent
+      link="body_hip_left" /><!--put 0.12 into -r to leg ||-->
     <child
       link="body_hip2_left" />
@@ -760,7 +760,7 @@
     <origin
       xyz="0.0006 0.11852 0.05341"
-      rpy="0.41 0 0" /><!--rpy="0 0 0" put -0.19 * -1 into r-->
-    <parent
-      link="leg2_left" /><!-- put 0.22 into r to prevent falling-->
+      rpy="0.41 0 0" /><!--rpy="0 0 0" put -0.19 into -r-->
+    <parent
+      link="leg2_left" /><!-- put -0.22 into -r to prevent falling-->
     <child
       link="leg3_left" />
@@ -819,5 +819,5 @@
     <origin
       xyz="-0.0241 -0.0065502 0.035907"
-      rpy="-2.9765 -0.0132 0.11369" /><!--rpy="-2.9765 -0.0732 0.41369" put 0.41 into p-->
+      rpy="-2.9765 -0.0132 0.03369" /><!--rpy="-2.9765 -0.0732 0.41369" put 0.41 into p-->
     <parent
       link="leg3_left" /><!-- and put -0.35 into p-->
@@ -825,5 +825,5 @@
       link="leg4_left" /><!-- and put -0.30 into y-->
     <axis
-      xyz="0 0 1" />
+      xyz="0 0 1" /><!--put 0.08 into -y to leg ||-->
     <dynamics
       damping="${dam}"
@@ -937,9 +937,9 @@
     <origin
       xyz="0.031042 0.015283 0.0465"
-      rpy="2.229 0 0.4575" /><!--rpy="1.479 0 0.4575" put -0.83 * -1 into r-->
-    <parent
-      link="body_hip_right" /><!-- and put -0.08 into r-->
-    <child
-      link="body_hip2_right" />
+      rpy="2.299 0 0.4575" /><!--rpy="1.479 0 0.4575" put -0.83 into -r-->
+    <parent
+      link="body_hip_right" /><!-- and put 0.08 into -r-->
+    <child
+      link="body_hip2_right" /><!--put -0.07 into -r to leg ||-->
     <axis
       xyz="-1 0 0" />
@@ -1173,5 +1173,5 @@
     <origin
       xyz="-0.0265 -0.035971 0.0061902"
-      rpy="1.753 -0.1059 3.1487" /><!--rpy="1.883 -0.9859 2.8787" put -1.08 into p-->
+      rpy="1.753 0.0141 3.1487" /><!--rpy="1.883 -0.9859 2.8787" put -1.08 into p-->
     <parent
       link="leg3_right" /><!-- and put 0.27 into y-->
@@ -1182,5 +1182,5 @@
     <dynamics
       damping="${dam}"
-      friction="${fri}" />
+      friction="${fri}" /><!--put -0.12 into -p to leg ||-->
     <limit
       effort="${lim_effort}"

Commit message: 爬起很稳，但走不动

File: dancer_urdf_model/robots/dancer_urdf_model.xacro (robot description, xacro)
@@ -14,6 +14,6 @@
   <xacro:property name="mass_lower" value="10.0"/><!--leg2,leg3,leg4-->
   <!--gazebo摩擦力-->
-  <xacro:property name="gazebo_mu1" value="0.8"/>
-  <xacro:property name="gazebo_mu2" value="0.8"/>
+  <xacro:property name="gazebo_mu1" value="0.4"/>
+  <xacro:property name="gazebo_mu2" value="0.4"/>
 <!-- root link -->
   <link
